File: badge/badge.kicad_pcb (KiCad board)
At the start: 2 copper layers, 73 x 68.6 mm, 56 parts, among them J1 USB_C_Receptacle_USB2.0, Q1 BSS138, Q2 BSS138, Q3 BSS138, Q4 BSS138, Q5 BC847BPN, SW1 Reset, SW2 Prog, U1 ESP-12F, U2 MDE029A128296RBW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

Commit message: Suff
Parts:
- added 3V3: Conn_01x01_Female, controls:Banana_THT, F.Cu at (95.2, 81.8)
- added GND: Conn_01x01_Female, controls:Banana_THT, F.Cu at (95.2, 76.2)
- added GP1: Conn_01x01_Female, controls:Banana_THT, F.Cu at (95.2, 87.4)
- added GP2: Conn_01x01_Female, controls:Banana_THT, F.Cu at (95.2, 93.0)
- added SCL: Conn_01x01_Female, controls:Banana_THT, F.Cu at (95.2, 104.1)
- added SDA: Conn_01x01_Female, controls:Banana_THT, F.Cu at (95.2, 98.6)
- moved G*** 30.5 mm to (64.5, 85.1) (x2)
- moved BT1 30.5 mm to (90.2, 114.3)
- moved C13 30.5 mm to (51.4, 114.3)
- moved C14 30.5 mm to (54.6, 116.8)
- moved D4 30.5 mm to (45.3, 109.2)
- moved D5 30.5 mm to (59.8, 106.7)
- moved D6 30.5 mm to (48.5, 109.2)
- moved D7 30.5 mm to (47.0, 109.2)
- moved Q2 30.5 mm to (45.5, 104.1)
- moved Q3 30.5 mm to (48.9, 104.1)
- moved Q4 30.5 mm to (41.9, 104.1)
- moved Q5 30.5 mm to (38.8, 99.9)
- moved R11 30.5 mm to (53.3, 106.7)
- moved R12 30.5 mm to (55.2, 106.7)
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Connections:
- net Net-(D5-Pad2) renamed /USB_P
- net Net-(D5-Pad3) renamed /USB_N
- C11 pad 1: Net-(C11-Pad1) -> Net-(3V3-Pad1)
- C12 pad 1: Net-(C11-Pad1) -> Net-(3V3-Pad1)
- L1 pad 1: Net-(C11-Pad1) -> Net-(3V3-Pad1)
- R1 pad 1: Net-(C11-Pad1) -> Net-(3V3-Pad1)
- R14 pad 1: Net-(D4-Pad2) -> Net-(CHG1-Pad2)
- R17 pad 1: Net-(D6-Pad2) -> Net-(R17-Pad1)
- R18 pad 1: Net-(D7-Pad2) -> Net-(R18-Pad1)
- R2 pad 1: Net-(C11-Pad1) -> Net-(3V3-Pad1)
- R3 pad 2: Net-(C11-Pad1) -> Net-(3V3-Pad1)
- R4 pad 1: Net-(C11-Pad1) -> Net-(3V3-Pad1)
- R5 pad 1: Net-(C11-Pad1) -> Net-(3V3-Pad1)
- R7 pad 1: Net-(C11-Pad1) -> Net-(3V3-Pad1)
- U1 pad 8: Net-(C11-Pad1) -> Net-(3V3-Pad1)
- U2 pad 15: Net-(C11-Pad1) -> Net-(3V3-Pad1)
- U2 pad 16: Net-(C11-Pad1) -> Net-(3V3-Pad1)
- U2 pad 8: Net-(C11-Pad1) -> Net-(3V3-Pad1)
- U3 pad 8: Net-(C11-Pad1) -> Net-(3V3-Pad1)
- U4 pad 5: Net-(C11-Pad1) -> Net-(3V3-Pad1)
- U5 pad 6: Net-(C11-Pad1) -> Net-(U5-Pad6)
- U5 pad 9: Net-(C11-Pad1) -> Net-(3V3-Pad1)
- U6 pad 1: Net-(D4-Pad1) -> Net-(CHG1-Pad1)
Routing:
- net Net-(3V3-Pad1): track 0.00 -> 244.2 mm, vias 0 -> 13
- net Net-(C11-Pad1): track 176.6 -> 0.00 mm, vias 12 -> 0
- net GND: track 287.6 -> 368.0 mm, vias 10 -> 11
- net Net-(R1-Pad2): track 74.4 -> 116.8 mm
- net Net-(GP2-Pad1): track 23.2 -> 61.5 mm, vias 1 -> 0
- net Net-(GP1-Pad1): track 11.2 -> 48.7 mm, vias 1 -> 2
- net Net-(U4-Pad6): track 8.37 -> 43.1 mm
- net Net-(U4-Pad7): track 7.94 -> 40.8 mm
- net Net-(U4-Pad10): track 24.1 -> 55.9 mm
- net Net-(R2-Pad2): track 70.1 -> 101.1 mm, vias 5 -> 4
- net Net-(U1-Pad22): track 94.3 -> 125.3 mm
- net Net-(Q5-Pad4): track 116.5 -> 147.5 mm
- net Net-(U1-Pad21): track 86.7 -> 117.6 mm
- net Net-(Q5-Pad6): track 113.0 -> 137.7 mm
- net Net-(U4-Pad8): track 32.5 -> 55.9 mm
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- removed copper zone on F.Cu, net (none)
Other:
- board size 73 x 68.6 mm -> 73 x 99.1 mm
