File: badge/badge.sch (KiCad schematic (older format))
At the start: 54 parts, among them J1 USB_C_Receptacle_USB2.0, Q1 BSS138, Q2 BSS138, Q3 BSS138, Q4 BSS138, Q5 BC847BPN, SW1 Reset, SW2 Prog, U1 ESP-12F, U2 MDE029A128296RBW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

Commit message: Suff
Parts:
- added 3V3, GND1, GP1, GP2, SCL1, SDA1: Conn_01x01_Female, Connector_PinHeader_1.00mm:PinHeader_1x01_P1.00mm_Vertical, symbol Connector:Conn_01x01_Female
- U2: symbol Custom~Parts:MDE029A128296RBW -> badge-rescue:MDE029A128296RBW-Custom_Parts
- U4: symbol Custom~Parts:CAP1296 -> badge-rescue:CAP1296-Custom_Parts
- U5: symbol Custom~Parts:CP2102N-A01-GQFN28_0 -> badge-rescue:CP2102N-A01-GQFN28_0-Custom_Parts
- renumbered CHG to CHG1, RX to RX1, TX to TX1
Connections:
- wire segments 335 -> 355
- no-connect marks 31 -> 29
Changed lines of the file:
@@
 EESchema Schematic File Version 4
+LIBS:badge-cache
 EELAYER 26 0
 EELAYER END
@@
 $EndDescr
 $Comp
-L Custom~Parts:MDE029A128296RBW U2
+L badge-rescue:MDE029A128296RBW-Custom_Parts U2
 U 1 1 5C3F7A34
 P 5650 1000
@@
 Connection ~ 7350 3550
 Wire Wire Line
-	7350 3550 7800 3550
+	7350 3550 7550 3550
 Wire Wire Line
 	7650 3350 7650 3450
 Connection ~ 7650 3450
 Wire Wire Line
-	7650 3450 6250 3450
+	7650 3450 7450 3450
 Wire Wire Line
 	7650 3050 7650 2850
@@
 Wire Wire Line
 	6100 1450 8950 1450
-NoConn ~ 6250 3650
 NoConn ~ 5050 3450
 Wire Wire Line
@@
 NoConn ~ 5050 4150
 $Comp
-L Custom~Parts:CAP1296 U4
+L badge-rescue:CAP1296-Custom_Parts U4
 U 1 1 5C53EF2E
 P 9950 3250
@@
 Wire Wire Line
 	5150 2050 5250 2050
-NoConn ~ 5050 3850
 Wire Wire Line
 	5150 2450 5150 2050
@@
 Connection ~ 7100 4450
 Wire Wire Line
-	7100 4450 8350 4450
+	7100 4450 7700 4450
 Wire Wire Line
 	7100 3700 6900 3700
@@
 Connection ~ 3550 2400
 $Comp
-L Custom~Parts:CP2102N-A01-GQFN28_0 U5
+L badge-rescue:CP2102N-A01-GQFN28_0-Custom_Parts U5
 U 1 1 5C8F01E4
 P 1450 3300
@@
 $EndComp
 $Comp
-L Device:LED CHG
+L Device:LED CHG1
 U 1 1 5CB2B8EB
 P 2450 900
-F 0 "CHG" H 2442 645 50  0000 C CNN
+F 0 "CHG1" H 2442 645 50  0000 C CNN
 F 1 "LED" H 2442 736 50  0000 C CNN
 F 2 "LED_SMD:LED_0603_1608Metric_Castellated" H 2450 900 50  0001 C CNN
@@
 Wire Wire Line
 	850  2700 850  2400
-Wire Wire Line
-	850  2400 1450 2400
 Connection ~ 1950 4450
 Wire Wire Line
@@
 Wire Wire Line
 	2400 2850 2400 2400
-Wire Wire Line
-	2400 2400 1450 2400
-Connection ~ 1450 2400
 NoConn ~ 2050 2700
 NoConn ~ 2050 2800
@@
 	2300 3800 2650 3800
 $Comp
-L Device:LED RX
+L Device:LED RX1
 U 1 1 5D3C9A2D
 P 3400 5400
-F 0 "RX" H 3392 5145 50  0000 C CNN
+F 0 "RX1" H 3392 5145 50  0000 C CNN
 F 1 "LED" H 3392 5236 50  0000 C CNN
 F 2 "LED_SMD:LED_0603_1608Metric_Castellated" H 3400 5400 50  0001 C CNN
@@
 $EndComp
 $Comp
-L Device:LED TX
+L Device:LED TX1
 U 1 1 5D3C9BA1
 P 3400 5750
-F 0 "TX" H 3392 5495 50  0000 C CNN
+F 0 "TX1" H 3392 5495 50  0000 C CNN
 F 1 "LED" H 3392 5586 50  0000 C CNN
 F 2 "LED_SMD:LED_0603_1608Metric_Castellated" H 3400 5750 50  0001 C CNN
@@
 Text Label 900  6150 0    50   ~ 0
 USB_N
+Wire Wire Line
+	850  2400 2400 2400
+$Comp
+L Connector:Conn_01x01_Female 3V3
+U 1 1 5C43DBF3
+P 8000 5000
+F 0 "3V3" H 8027 5026 50  0000 L CNN
+F 1 "Conn_01x01_Female" H 8027 4935 50  0000 L CNN
+F 2 "Connector_PinHeader_1.00mm:PinHeader_1x01_P1.00mm_Vertical" H 8000 5000 50  0001 C CNN
+F 3 "~" H 8000 5000 50  0001 C CNN
+	1    8000 5000
+	1    0    0    -1
+$EndComp
+$Comp
+L Connector:Conn_01x01_Female GND1
+U 1 1 5C43DD01
+P 8000 5150
+F 0 "GND1" H 8027 5176 50  0000 L CNN
+F 1 "Conn_01x01_Female" H 8027 5085 50  0000 L CNN
+F 2 "Connector_PinHeader_1.00mm:PinHeader_1x01_P1.00mm_Vertical" H 8000 5150 50  0001 C CNN
+F 3 "~" H 8000 5150 50  0001 C CNN
+	1    8000 5150
+	1    0    0    -1
+$EndComp
+$Comp
+L Connector:Conn_01x01_Female GP1
+U 1 1 5C43DDF4
+P 8000 5300
+F 0 "GP1" H 8027 5326 50  0000 L CNN
+F 1 "Conn_01x01_Female" H 8027 5235 50  0000 L CNN
+F 2 "Connector_PinHeader_1.00mm:PinHeader_1x01_P1.00mm_Vertical" H 8000 5300 50  0001 C CNN
+F 3 "~" H 8000 5300 50  0001 C CNN
+	1    8000 5300
+	1    0    0    -1
+$EndComp
+$Comp
+L Connector:Conn_01x01_Female GP2
+U 1 1 5C43DECA
+P 8000 5450
+F 0 "GP2" H 8027 5476 50  0000 L CNN
+F 1 "Conn_01x01_Female" H 8027 5385 50  0000 L CNN
+F 2 "Connector_PinHeader_1.00mm:PinHeader_1x01_P1.00mm_Vertical" H 8000 5450 50  0001 C CNN
+F 3 "~" H 8000 5450 50  0001 C CNN
+	1    8000 5450
+	1    0    0    -1
+$EndComp
+$Comp
+L Connector:Conn_01x01_Female SCL1
+U 1 1 5C43DFA3
+P 8000 5600
+F 0 "SCL1" H 8027 5626 50  0000 L CNN
+F 1 "Conn_01x01_Female" H 8027 5535 50  0000 L CNN
+F 2 "Connector_PinHeader_1.00mm:PinHeader_1x01_P1.00mm_Vertical" H 8000 5600 50  0001 C CNN
+F 3 "~" H 8000 5600 50  0001 C CNN
+	1    8000 5600
+	1    0    0    -1
+$EndComp
+$Comp
+L Connector:Conn_01x01_Female SDA1
+U 1 1 5C43E083
+P 8000 5750
+F 0 "SDA1" H 8027 5776 50  0000 L CNN
+F 1 "Conn_01x01_Female" H 8027 5685 50  0000 L CNN
+F 2 "Connector_PinHeader_1.00mm:PinHeader_1x01_P1.00mm_Vertical" H 8000 5750 50  0001 C CNN
+F 3 "~" H 8000 5750 50  0001 C CNN
+	1    8000 5750
+	1    0    0    -1
+$EndComp
+Wire Wire Line
+	7200 3350 7200 3500
+Wire Wire Line
+	7200 3500 7750 3500
+Wire Wire Line
+	7750 3500 7750 5000
+Wire Wire Line
+	7750 5000 7800 5000
+Connection ~ 7200 3350
+Wire Wire Line
+	7800 5150 7700 5150
+Wire Wire Line
+	7700 5150 7700 4450
+Connection ~ 7700 4450
+Wire Wire Line
+	7700 4450 8350 4450
+Wire Wire Line
+	5050 3850 4950 3850
+Wire Wire Line
+	4950 3850 4950 4550
+Wire Wire Line
+	4950 4550 7650 4550
+Wire Wire Line
+	7650 4550 7650 5300
+Wire Wire Line
+	7650 5300 7800 5300
+Wire Wire Line
+	7800 5450 7600 5450
+Wire Wire Line
+	7600 5450 7600 3650
+Wire Wire Line
+	7600 3650 6250 3650
+Wire Wire Line
+	7550 3550 7550 5600
+Wire Wire Line
+	7550 5600 7800 5600
+Connection ~ 7550 3550
+Wire Wire Line
+	7550 3550 7800 3550
+Wire Wire Line
+	7450 3450 7450 5750
+Wire Wire Line
+	7450 5750 7800 5750
+Connection ~ 7450 3450
+Wire Wire Line
+	7450 3450 6250 3450
 $EndSCHEMATC
